File: trunk/schematics/HomeAutomation/AVR/nodes/obdNode/obdNode.sch (EAGLE design)
At the start: 30 parts, among them IC1 MCP2515, IC2 TH8056KDC-AAA-008-RE, IC3 AMIS42665, IC4 ATMEGA64-TQFP32TQFP32, IC5 LM2674, X1 AVRISP6PINHEADER, X2 MICROMATCH-6

Commit message: Work on obdNode
git-svn-id: http://svn.arune.se/svn/hardware@888 bbe6898a-5d1e-0410-8d97-fea9c15d82f3
Parts:
- added C4: 100n, rcl:C-EUC0402
- R1, R4: value 10k -> (none)
Connections:
- net GND: now also C4.2
- net VBAT: now also C4.1
Other:
- moved on the sheet: R3
Changed lines of the file:
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@@
 <?xml version="1.0" encoding="utf-8"?>
 <!DOCTYPE eagle SYSTEM "eagle.dtd">
-<eagle version="6.4">
+<eagle version="6.5.0">
 <drawing>
 <settings>
@@
 <part name="C13" library="rcl" deviceset="C-EU" device="C0402" value="100n"/>
 <part name="V17" library="supply2" deviceset="VCC" device=""/>
-<part name="R1" library="rcl" deviceset="R-EU" device="R0402" value="10k"/>
+<part name="R1" library="rcl" deviceset="R-EU" device="R0402"/>
 <part name="V18" library="supply2" deviceset="VCC" device=""/>
 <part name="V19" library="supply2" deviceset="GND" device=""/>
@@
 <part name="D4" library="diode" deviceset="DUALTVS" device="SOT23" value="NUP2105L"/>
 <part name="V20" library="supply2" deviceset="GND" device=""/>
-<part name="R4" library="rcl" deviceset="R-EU" device="R0402" value="10k"/>
+<part name="R4" library="rcl" deviceset="R-EU" device="R0402"/>
 <part name="V21" library="supply2" deviceset="VCC" device=""/>
 <part name="V22" library="supply2" deviceset="GND" device=""/>
 <part name="Q1" library="xtal_CSTCE" deviceset="CSTCE" device="SMD"/>
+<part name="C4" library="rcl" deviceset="C-EU" device="C0402" value="100n"/>
 </parts>
 <sheets>
@@
 <attribute name="VALUE" x="-17.78" y="-68.58" size="1.778" layer="96"/>
 </instance>
-<instance part="R3" gate="R" x="10.16" y="-53.34" rot="R90"/>
+<instance part="R3" gate="R" x="7.62" y="-53.34" rot="R90"/>
 <instance part="V16" gate="GND" x="5.08" y="-63.5" smashed="yes">
 <attribute name="VALUE" x="3.175" y="-66.675" size="1.778" layer="96"/>
@@
 <instance part="V22" gate="GND" x="-55.88" y="-7.62"/>
 <instance part="Q1" gate="G$1" x="-55.88" y="2.54"/>
+<instance part="C4" gate="C" x="27.94" y="78.74"/>
 </instances>
 <busses>
@@
 <pinref part="C42" gate="C" pin="2"/>
 <pinref part="C41" gate="C" pin="2"/>
+<pinref part="C4" gate="C" pin="2"/>
+<wire x1="27.94" y1="73.66" x2="27.94" y2="71.12" width="0.1524" layer="91"/>
+<wire x1="27.94" y1="71.12" x2="35.56" y2="71.12" width="0.1524" layer="91"/>
+<junction x="35.56" y="71.12"/>
 </segment>
 <segment>
@@
 </segment>
 <segment>
-<wire x1="35.56" y1="86.36" x2="35.56" y2="81.28" width="0.1524" layer="91"/>
+<wire x1="35.56" y1="86.36" x2="35.56" y2="83.82" width="0.1524" layer="91"/>
 <label x="35.56" y="86.36" size="1.778" layer="95"/>
 <pinref part="C41" gate="C" pin="1"/>
+<pinref part="C4" gate="C" pin="1"/>
+<wire x1="35.56" y1="83.82" x2="35.56" y2="81.28" width="0.1524" layer="91"/>
+<wire x1="27.94" y1="81.28" x2="27.94" y2="83.82" width="0.1524" layer="91"/>
+<wire x1="27.94" y1="83.82" x2="35.56" y2="83.82" width="0.1524" layer="91"/>
+<junction x="35.56" y="83.82"/>
 </segment>
 <segment>
@@
 </segment>
 <segment>
-<wire x1="15.24" y1="-48.26" x2="10.16" y2="-48.26" width="0.1524" layer="91"/>
-<wire x1="10.16" y1="-48.26" x2="2.54" y2="-48.26" width="0.1524" layer="91"/>
+<wire x1="15.24" y1="-48.26" x2="7.62" y2="-48.26" width="0.1524" layer="91"/>
+<wire x1="7.62" y1="-48.26" x2="2.54" y2="-48.26" width="0.1524" layer="91"/>
 <wire x1="15.24" y1="-50.8" x2="15.24" y2="-48.26" width="0.1524" layer="91"/>
-<junction x="10.16" y="-48.26"/>
+<junction x="7.62" y="-48.26"/>
 <label x="15.24" y="-48.26" size="1.778" layer="95"/>
 <pinref part="IC2" gate="MCP2551" pin="CANH"/>
@@
 <net name="N$3" class="0">
 <segment>
-<wire x1="10.16" y1="-58.42" x2="5.08" y2="-58.42" width="0.1524" layer="91"/>
-<wire x1="5.08" y1="-58.42" x2="5.08" y2="-55.88" width="0.1524" layer="91"/>
-<wire x1="5.08" y1="-55.88" x2="2.54" y2="-55.88" width="0.1524" layer="91"/>
+<wire x1="7.62" y1="-58.42" x2="2.54" y2="-58.42" width="0.1524" layer="91"/>
+<wire x1="2.54" y1="-58.42" x2="2.54" y2="-55.88" width="0.1524" layer="91"/>
 <pinref part="R3" gate="R" pin="1"/>
 <pinref part="IC2" gate="MCP2551" pin="LOAD"/>
