File: trunk/schematics/HomeAutomation/AVR/nodes/hpdNode/hpdNode.brd (EAGLE design)
At the start: 32.8 x 23.2 mm, 34 parts, among them IC1 MCP2515, IC2 AMIS42665, IC3 ATMEGA88-M32, IC4 AMIS42665, IC5 BD9G101G, X2 AVRISP6PINHEADER

Commit message: Schematic done
git-svn-id: http://svn.arune.se/svn/hardware@898 bbe6898a-5d1e-0410-8d97-fea9c15d82f3
Parts:
- removed D5: NUP2105L, diode:SOT23
- added C14, C15, C16, C17: 100n, rcl:C0402
- added IC6, IC7, IC8: TS5A3167DBV, ts5a3167:SOT23-5
- added IC9: LT1129IS8-5, lt1129:SO8
- added R3, R4, R5: (no value), rcl:R0402
- C1: value 100n -> 10n/100V; device rcl:C0402 -> rcl:C0805
- C4: value 100n -> 3u3/50V; device rcl:C0402 -> rcl:C1210
- moved D4 68.5 mm to (47.1, 43.7)
- moved IC4 31.5 mm to (18.8, 47.2)
- moved C3 15.8 mm to (53.3, 18.3)
- moved IC2 13.4 mm to (12.8, 47.2), turned to 0 degrees
- moved X2 12.4 mm to (4.19, 38.5), turned to 270 degrees
- moved C1 12.2 mm to (64.0, 33.5)
- moved C10 8.24 mm to (12.7, 43.3), turned to 180 degrees
- moved JP1 6.86 mm to (26.4, 55.4)
- moved C2 5.88 mm to (48.9, 18.5)
- moved C4 5.23 mm to (-0.51, -14.7)
- moved JP2 2.82 mm to (24.9, 22.6)
- moved C13 1.65 mm to (18.5, 33.9)
- moved C41 1.65 mm to (35.2, 33.1)
- moved D1 1.65 mm to (35.9, 36.2)
- moved C11 1.65 mm to (26.2, 33.8)
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Connections:
- new net EXP_O: IC3.24, IC9.5
- net EXP_E: now also IC8.4, R3.2
- net EXP_F: now also IC7.4, R4.2
- net EXP_G: now also IC6.4, R5.2
- net GND: now also C14.2, C15.2, C16.2, C17.2, IC6.3, IC7.3, IC8.3, IC9.3, IC9.6, IC9.7, R3.1, R4.1, R5.1; no longer D5.3
- net UARTH_IN: now also IC6.1; no longer D5.2
- net UARTH_OUT: now also IC6.2
- net UARTL_IN: now also IC7.1; no longer D5.1
- net UARTL_OUT: now also IC7.2
- net VCC: now also C14.1, C15.1, C16.1, C17.1, IC6.5, IC7.5, IC8.5; no longer C1.1, C4.1
- net V_CAN: now also IC9.8
- net WAKE_IN: now also IC8.1
- net WAKE_OUT: now also C1.1, C4.1, IC8.2, IC9.1, IC9.2; no longer IC3.24
Routing:
- net RXCAN: track 19.3 -> 2.21 mm, vias 2 -> 0
- net TXCAN: track 12.3 -> 0.34 mm
- net GND: track 35.2 -> 33.3 mm
- net VCC: track 52.2 -> 50.2 mm
- net EXP_O: track 0.00 -> 1.88 mm, vias 0 -> 1
- net WAKE_OUT: track 1.88 -> 0.00 mm, vias 1 -> 0
Other:
- board size 32.8 x 23.2 mm -> 34.9 x 43.9 mm
