File: trunk/schematics/HomeAutomation/AVR/nodes/hpdNode/hpdNode.sch (EAGLE design)
At the start: 34 parts, among them IC1 MCP2515, IC2 AMIS42665, IC3 ATMEGA88-M32, IC4 AMIS42665, IC5 BD9G101G, X2 AVRISP6PINHEADER

Commit message: Schematic done
git-svn-id: http://svn.arune.se/svn/hardware@898 bbe6898a-5d1e-0410-8d97-fea9c15d82f3
Parts:
- removed D5: NUP2105L, diode:DUALTVSSOT23
- added C14, C15, C16, C17: 100n, rcl:C-EUC0402
- added IC6, IC7, IC8: TS5A3167DBV, ts5a3167:TS5A3167DBV
- added IC9: LT1129IS8-5, lt1129:LT1129-5SO8
- added R3, R4, R5: (no value), rcl:R-EUR0402
- C1: value 100n -> 10n/100V; device rcl:C-EUC0402 -> rcl:C-EUC0805
- C4: value 100n -> 3u3/50V; device rcl:C-EUC0402 -> rcl:C-EUC1210
Connections:
- new net EXP_O: IC3.PC1(ADC1/PCINT9), IC9.SHDN
- net EXP_E: now also IC8.IN, R3.2
- net EXP_F: now also IC7.IN, R4.2
- net EXP_G: now also IC6.IN, R5.2
- net GND: now also C14.2, C15.2, C16.2, C17.2, IC6.GND, IC7.GND, IC8.GND, IC9.GND, IC9.GND1, IC9.GND2, R3.1, R4.1, R5.1; no longer D5.3
- net UARTH_IN: now also IC6.NC; no longer D5.2
- net UARTH_OUT: now also IC6.COM
- net UARTL_IN: now also IC7.NC; no longer D5.1
- net UARTL_OUT: now also IC7.COM
- net VCC: now also C14.1, C15.1, C16.1, C17.1, IC6.VCC, IC7.VCC, IC8.VCC; no longer C1.1, C4.1
- net V_CAN: now also IC9.IN
- net WAKE_IN: now also IC8.NC
- net WAKE_OUT: now also C1.1, C4.1, IC8.COM, IC9.OUT, IC9.SENSE; no longer IC3.PC1(ADC1/PCINT9)
Other:
- note added: "INCOMING FROM CAR"
- note added: "OUTGOING TO DISPLAY"
- note added: "Reverse polarity protection"
- note removed: "FROM CAR"
- note removed: "INCOMING"
- note removed: "OUTGOING"
- note removed: "Reverse"
- note removed: "TO DISPLAY"
- note removed: "polarity"
- note removed: "protection"
- moved on the sheet: C1, C10, C11, C12, C13, C2, C3, C4, C40, C44, D1, D2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
